File: Hardware/Prebuilt_Module/Version_1.0/Schematic_start_module_sumo_IR_V1_0.sch (EAGLE design)
At the start: 19 parts, among them IC1 ATTINY24,44,84_QFNVQFN

Commit message: Some corrections from 1.0
Due to some errors, I decided to switch to 0402 components, thus making
it easier to route and to add another feature: a serial resistor for
the home-pad. The signals for the pads used for the pogo-bead are
changed. The positions are still the same, but the signals are a little
mixed.
Parts:
- added R6: 1k, rcl:R-EU_R0402
- MISO_PAD: value (none) -> mosi
- MOSI_PAD: value mosi -> (none); device CRF:PAD75X75 -> CRF:PAD50X50
- R1, R2, R3, R4, R5: device rcl:R-EU_R0603 -> rcl:R-EU_R0402
- SCK_PAD: device CRF:PAD50X50 -> CRF:PAD75X75
- renumbered C3 to C2
Connections:
- removed net LED: IC1.PA7(ADC7/ISCP/OC0B), R2.2
- new net KILL: IC1.PA7(ADC7/ISCP/OC0B), R5.1
- new net N$2: R6.1, SCK_PAD.PAD
- new net START: IC1.PB2(INT0/OC0A), R3.1
- net GND: now also LED.C
- net IR: now also IC1.PA0(ADC0/AREF); no longer IC1.PB0(CLKI/XTAL1)
- net MISO: now also R2.2
- net MOSI: no longer R3.1
- net N$1: now also LED.A; no longer LED.C
- net SCK: now also R6.2; no longer R5.1, SCK_PAD.PAD
- net VCC: no longer LED.A
Other:
- moved on the sheet: LED, MISO_PAD, MOSI_PAD, R3, R5
